File: Common_ERR.kicad_sch (KiCad schematic)
At the start: 5 parts

Commit message: Изменил схему
Parts:
- removed C25, C26: 2.2u, Capacitor_SMD:C_0805_2012Metric_Pad1.18x1.45mm_HandSolder, symbol Device:C_Small
- removed D10: SN74HC11DR, Package_SO:SOIC-14_3.9x8.7mm_P1.27mm, symbol Logic_My:SN74HC11DR
- removed D11: ADM3485E, Package_SO:SOIC-8_3.9x4.9mm_P1.27mm, symbol Interface_My:ADM3485E
- removed R36: 120, Resistor_SMD:R_0805_2012Metric_Pad1.20x1.40mm_HandSolder, symbol Device:R_Small
Connections:
- no-connect marks 9 -> 0
