File: Fault2.kicad_sch (KiCad schematic)
At the start: 26 parts

Commit message: Изменил схему
Parts:
- removed C10, C11, C12, C9: 56p, Capacitor_SMD:C_0805_2012Metric_Pad1.18x1.45mm_HandSolder, symbol Device:C_Small
- removed C37: 2.2u, Capacitor_SMD:C_0805_2012Metric_Pad1.18x1.45mm_HandSolder, symbol Device:C_Small
- removed D4: SN74AC08DR, Package_SO:SOIC-14_3.9x8.7mm_P1.27mm, symbol Logic:SN74AC08DR
- removed R5, R6, R7, R8: 120, Resistor_SMD:R_0805_2012Metric_Pad1.20x1.40mm_HandSolder, symbol Device:R_Small
- R47, R49: value 10k -> 30k
- R48, R51: value 120 -> 30k
Connections:
- no-connect marks 3 -> 0
