File: NTC_Reset_A.kicad_sch (KiCad schematic)
At the start: 8 parts, among them U3 LMV331

Commit message: Убрал питание 3.3В
Connections:
- net +3V3 renamed +5V
Changed lines of the file:
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@@
 	)
 	(symbol
-		(lib_id "power:+3.3V")
+		(lib_id "power:+5V")
 		(at 139.065 95.25 0)
 		(unit 1)
@@
 		(on_board yes)
 		(dnp no)
-		(property "Reference" "#PWR063"
+		(property "Reference" "#PWR63"
 			(at 139.065 99.06 0)
 			(effects
@@
 			)
 		)
-		(property "Value" "+3V3"
-			(at 139.065 92.075 0)
+		(property "Value" "+5V"
+			(at 139.065 91.694 0)
 			(effects
 				(font
@@
 			)
 		)
-		(property "Description" ""
+		(property "Description" "Power symbol creates a global label with name \"+5V\""
 			(at 139.065 95.25 0)
 			(effects
@@
 			(project "Adapter"
 				(path "/e63e39d7-6ac0-4ffd-8aa3-1841a4541b55/58345529-7f56-4564-b4a1-0045dc902a9f"
-					(reference "#PWR063")
-					(unit 1)
-				)
-			)
-		)
-	)
-	(symbol
-		(lib_id "power:+3.3V")
+					(reference "#PWR63")
+					(unit 1)
+				)
+			)
+		)
+	)
+	(symbol
+		(lib_id "power:+5V")
 		(at 121.92 95.885 0)
 		(unit 1)
@@
 		(on_board yes)
 		(dnp no)
-		(property "Reference" "#PWR066"
+		(property "Reference" "#PWR66"
 			(at 121.92 99.695 0)
 			(effects
@@
 			)
 		)
-		(property "Value" "+3V3"
-			(at 121.92 91.44 0)
+		(property "Value" "+5V"
+			(at 121.92 92.329 0)
 			(effects
 				(font
@@
 			)
 		)
-		(property "Description" ""
+		(property "Description" "Power symbol creates a global label with name \"+5V\""
 			(at 121.92 95.885 0)
 			(effects
@@
 			(project "Adapter"
 				(path "/e63e39d7-6ac0-4ffd-8aa3-1841a4541b55/58345529-7f56-4564-b4a1-0045dc902a9f"
-					(reference "#PWR066")
+					(reference "#PWR66")
 					(unit 1)
 				)
@@
 	)
 	(symbol
-		(lib_id "power:+3.3V")
+		(lib_id "power:+5V")
 		(at 155.575 95.25 0)
 		(unit 1)
@@
 		(on_board yes)
 		(dnp no)
-		(property "Reference" "#PWR064"
+		(property "Reference" "#PWR64"
 			(at 155.575 99.06 0)
 			(effects
@@
 			)
 		)
-		(property "Value" "+3V3"
-			(at 155.575 92.075 0)
+		(property "Value" "+5V"
+			(at 155.575 91.694 0)
 			(effects
 				(font
@@
 			)
 		)
-		(property "Description" ""
+		(property "Description" "Power symbol creates a global label with name \"+5V\""
 			(at 155.575 95.25 0)
 			(effects
@@
 			(project "Adapter"
 				(path "/e63e39d7-6ac0-4ffd-8aa3-1841a4541b55/58345529-7f56-4564-b4a1-0045dc902a9f"
-					(reference "#PWR064")
-					(unit 1)
-				)
-			)
-		)
-	)
-	(symbol
-		(lib_id "power:+3.3V")
+					(reference "#PWR64")
+					(unit 1)
+				)
+			)
+		)
+	)
+	(symbol
+		(lib_id "power:+5V")
 		(at 116.205 112.395 180)
 		(unit 1)
@@
 		(on_board yes)
 		(dnp no)
-		(property "Reference" "#PWR068"
+		(property "Reference" "#PWR68"
 			(at 116.205 108.585 0)
 			(effects
@@
 			)
 		)
-		(property "Value" "+3V3"
-			(at 116.205 116.84 0)
+		(property "Value" "+5V"
+			(at 116.205 115.951 0)
 			(effects
 				(font
@@
 			)
 		)
-		(property "Description" ""
+		(property "Description" "Power symbol creates a global label with name \"+5V\""
 			(at 116.205 112.395 0)
 			(effects
@@
 			(project "Adapter"
 				(path "/e63e39d7-6ac0-4ffd-8aa3-1841a4541b55/58345529-7f56-4564-b4a1-0045dc902a9f"
-					(reference "#PWR068")
+					(reference "#PWR68")
 					(unit 1)
 				)
@@
 	)
 	(symbol
-		(lib_id "power:+3.3V")
+		(lib_id "power:+5V")
 		(at 139.065 78.105 0)
 		(unit 1)
@@
 		(on_board yes)
 		(dnp no)
-		(property "Reference" "#PWR061"
+		(property "Reference" "#PWR61"
 			(at 139.065 81.915 0)
 			(effects
@@
 			)
 		)
-		(property "Value" "+3V3"
-			(at 139.065 74.93 0)
+		(property "Value" "+5V"
+			(at 139.065 74.549 0)
 			(effects
 				(font
@@
 			)
 		)
-		(property "Description" ""
+		(property "Description" "Power symbol creates a global label with name \"+5V\""
 			(at 139.065 78.105 0)
 			(effects
@@
 			(project "Adapter"
 				(path "/e63e39d7-6ac0-4ffd-8aa3-1841a4541b55/58345529-7f56-4564-b4a1-0045dc902a9f"
-					(reference "#PWR061")
-					(unit 1)
-				)
+					(reference "#PWR61")
+					(unit 1)
+				)
