File: NTC_Reset_B.kicad_sch (KiCad schematic)
At the start: 8 parts, among them U4 LMV331

Commit message: Убрал питание 3.3В
Connections:
- net +3V3 renamed +5V
Changed lines of the file:
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@@
 	)
 	(symbol
-		(lib_id "power:+3.3V")
+		(lib_id "power:+5V")
 		(at 121.92 95.885 0)
 		(unit 1)
@@
 		(on_board yes)
 		(dnp no)
-		(property "Reference" "#PWR082"
+		(property "Reference" "#PWR82"
 			(at 121.92 99.695 0)
 			(effects
@@
 			)
 		)
-		(property "Value" "+3V3"
-			(at 121.92 91.44 0)
+		(property "Value" "+5V"
+			(at 121.92 92.329 0)
 			(effects
 				(font
@@
 			)
 		)
-		(property "Description" ""
+		(property "Description" "Power symbol creates a global label with name \"+5V\""
 			(at 121.92 95.885 0)
 			(effects
@@
 			(project "Adapter"
 				(path "/e63e39d7-6ac0-4ffd-8aa3-1841a4541b55/83a29e8e-3522-4bfb-8d85-061a14678ae9"
-					(reference "#PWR082")
+					(reference "#PWR82")
 					(unit 1)
 				)
@@
 	)
 	(symbol
-		(lib_id "power:+3.3V")
+		(lib_id "power:+5V")
 		(at 116.205 112.395 180)
 		(unit 1)
@@
 		(on_board yes)
 		(dnp no)
-		(property "Reference" "#PWR084"
+		(property "Reference" "#PWR84"
 			(at 116.205 108.585 0)
 			(effects
@@
 			)
 		)
-		(property "Value" "+3V3"
-			(at 116.205 116.84 0)
+		(property "Value" "+5V"
+			(at 116.205 115.951 0)
 			(effects
 				(font
@@
 			)
 		)
-		(property "Description" ""
+		(property "Description" "Power symbol creates a global label with name \"+5V\""
 			(at 116.205 112.395 0)
 			(effects
@@
 			(project "Adapter"
 				(path "/e63e39d7-6ac0-4ffd-8aa3-1841a4541b55/83a29e8e-3522-4bfb-8d85-061a14678ae9"
-					(reference "#PWR084")
+					(reference "#PWR84")
 					(unit 1)
 				)
@@
 	)
 	(symbol
-		(lib_id "power:+3.3V")
+		(lib_id "power:+5V")
 		(at 155.575 95.25 0)
 		(unit 1)
@@
 		(on_board yes)
 		(dnp no)
-		(property "Reference" "#PWR079"
+		(property "Reference" "#PWR79"
 			(at 155.575 99.06 0)
 			(effects
@@
 			)
 		)
-		(property "Value" "+3V3"
-			(at 155.575 92.075 0)
+		(property "Value" "+5V"
+			(at 155.575 91.694 0)
 			(effects
 				(font
@@
 			)
 		)
-		(property "Description" ""
+		(property "Description" "Power symbol creates a global label with name \"+5V\""
 			(at 155.575 95.25 0)
 			(effects
@@
 			(project "Adapter"
 				(path "/e63e39d7-6ac0-4ffd-8aa3-1841a4541b55/83a29e8e-3522-4bfb-8d85-061a14678ae9"
-					(reference "#PWR079")
+					(reference "#PWR79")
 					(unit 1)
 				)
@@
 	)
 	(symbol
-		(lib_id "power:+3.3V")
+		(lib_id "power:+5V")
 		(at 139.065 78.105 0)
 		(unit 1)
@@
 		(on_board yes)
 		(dnp no)
-		(property "Reference" "#PWR072"
+		(property "Reference" "#PWR72"
 			(at 139.065 81.915 0)
 			(effects
@@
 			)
 		)
-		(property "Value" "+3V3"
-			(at 139.065 74.93 0)
+		(property "Value" "+5V"
+			(at 139.065 74.549 0)
 			(effects
 				(font
@@
 			)
 		)
-		(property "Description" ""
+		(property "Description" "Power symbol creates a global label with name \"+5V\""
 			(at 139.065 78.105 0)
 			(effects
@@
 			(project "Adapter"
 				(path "/e63e39d7-6ac0-4ffd-8aa3-1841a4541b55/83a29e8e-3522-4bfb-8d85-061a14678ae9"
-					(reference "#PWR072")
+					(reference "#PWR72")
 					(unit 1)
 				)
@@
 	)
 	(symbol
-		(lib_id "power:+3.3V")
+		(lib_id "power:+5V")
 		(at 139.065 95.25 0)
 		(unit 1)
@@
 		(on_board yes)
 		(dnp no)
-		(property "Reference" "#PWR076"
+		(property "Reference" "#PWR76"
 			(at 139.065 99.06 0)
 			(effects
@@
 			)
 		)
-		(property "Value" "+3V3"
-			(at 139.065 92.075 0)
+		(property "Value" "+5V"
+			(at 139.065 91.694 0)
 			(effects
 				(font
@@
 			)
 		)
-		(property "Description" ""
+		(property "Description" "Power symbol creates a global label with name \"+5V\""
 			(at 139.065 95.25 0)
 			(effects
@@
 			(project "Adapter"
 				(path "/e63e39d7-6ac0-4ffd-8aa3-1841a4541b55/83a29e8e-3522-4bfb-8d85-061a14678ae9"
-					(reference "#PWR076")
-					(unit 1)
-				)
+					(reference "#PWR76")
+					(unit 1)
+				)
