File: NTC_Reset_C.kicad_sch (KiCad schematic)
At the start: 8 parts, among them U6 LMV331

Commit message: Убрал питание 3.3В
Connections:
- net +3V3 renamed +5V
Changed lines of the file:
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@@
 	)
 	(symbol
-		(lib_id "power:+3.3V")
+		(lib_id "power:+5V")
 		(at 121.92 95.885 0)
 		(unit 1)
@@
 		(on_board yes)
 		(dnp no)
-		(property "Reference" "#PWR093"
+		(property "Reference" "#PWR93"
 			(at 121.92 99.695 0)
 			(effects
@@
 			)
 		)
-		(property "Value" "+3V3"
-			(at 121.92 91.44 0)
+		(property "Value" "+5V"
+			(at 121.92 92.329 0)
 			(effects
 				(font
@@
 			)
 		)
-		(property "Description" ""
+		(property "Description" "Power symbol creates a global label with name \"+5V\""
 			(at 121.92 95.885 0)
 			(effects
@@
 			(project "Adapter"
 				(path "/e63e39d7-6ac0-4ffd-8aa3-1841a4541b55/7f3c60e8-60b4-472a-9873-5fab779b18b2"
-					(reference "#PWR093")
-					(unit 1)
-				)
-			)
-		)
-	)
-	(symbol
-		(lib_id "power:+3.3V")
+					(reference "#PWR93")
+					(unit 1)
+				)
+			)
+		)
+	)
+	(symbol
+		(lib_id "power:+5V")
 		(at 139.065 78.105 0)
 		(unit 1)
@@
 		(on_board yes)
 		(dnp no)
-		(property "Reference" "#PWR088"
+		(property "Reference" "#PWR88"
 			(at 139.065 81.915 0)
 			(effects
@@
 			)
 		)
-		(property "Value" "+3V3"
-			(at 139.065 74.93 0)
+		(property "Value" "+5V"
+			(at 139.065 74.549 0)
 			(effects
 				(font
@@
 			)
 		)
-		(property "Description" ""
+		(property "Description" "Power symbol creates a global label with name \"+5V\""
 			(at 139.065 78.105 0)
 			(effects
@@
 			(project "Adapter"
 				(path "/e63e39d7-6ac0-4ffd-8aa3-1841a4541b55/7f3c60e8-60b4-472a-9873-5fab779b18b2"
-					(reference "#PWR088")
+					(reference "#PWR88")
 					(unit 1)
 				)
@@
 	)
 	(symbol
-		(lib_id "power:+3.3V")
+		(lib_id "power:+5V")
 		(at 139.065 95.25 0)
 		(unit 1)
@@
 		(on_board yes)
 		(dnp no)
-		(property "Reference" "#PWR090"
+		(property "Reference" "#PWR90"
 			(at 139.065 99.06 0)
 			(effects
@@
 			)
 		)
-		(property "Value" "+3V3"
-			(at 139.065 92.075 0)
+		(property "Value" "+5V"
+			(at 139.065 91.694 0)
 			(effects
 				(font
@@
 			)
 		)
-		(property "Description" ""
+		(property "Description" "Power symbol creates a global label with name \"+5V\""
 			(at 139.065 95.25 0)
 			(effects
@@
 			(project "Adapter"
 				(path "/e63e39d7-6ac0-4ffd-8aa3-1841a4541b55/7f3c60e8-60b4-472a-9873-5fab779b18b2"
-					(reference "#PWR090")
+					(reference "#PWR90")
 					(unit 1)
 				)
@@
 	)
 	(symbol
-		(lib_id "power:+3.3V")
+		(lib_id "power:+5V")
 		(at 116.205 112.395 180)
 		(unit 1)
@@
 		(on_board yes)
 		(dnp no)
-		(property "Reference" "#PWR095"
+		(property "Reference" "#PWR95"
 			(at 116.205 108.585 0)
 			(effects
@@
 			)
 		)
-		(property "Value" "+3V3"
-			(at 116.205 116.84 0)
+		(property "Value" "+5V"
+			(at 116.205 115.951 0)
 			(effects
 				(font
@@
 			)
 		)
-		(property "Description" ""
+		(property "Description" "Power symbol creates a global label with name \"+5V\""
 			(at 116.205 112.395 0)
 			(effects
@@
 			(project "Adapter"
 				(path "/e63e39d7-6ac0-4ffd-8aa3-1841a4541b55/7f3c60e8-60b4-472a-9873-5fab779b18b2"
-					(reference "#PWR095")
+					(reference "#PWR95")
 					(unit 1)
 				)
@@
 	)
 	(symbol
-		(lib_id "power:+3.3V")
+		(lib_id "power:+5V")
 		(at 155.575 95.25 0)
 		(unit 1)
@@
 		(on_board yes)
 		(dnp no)
-		(property "Reference" "#PWR091"
+		(property "Reference" "#PWR91"
 			(at 155.575 99.06 0)
 			(effects
@@
 			)
 		)
-		(property "Value" "+3V3"
-			(at 155.575 92.075 0)
+		(property "Value" "+5V"
+			(at 155.575 91.694 0)
 			(effects
 				(font
@@
 			)
 		)
-		(property "Description" ""
+		(property "Description" "Power symbol creates a global label with name \"+5V\""
 			(at 155.575 95.25 0)
 			(effects
@@
 			(project "Adapter"
 				(path "/e63e39d7-6ac0-4ffd-8aa3-1841a4541b55/7f3c60e8-60b4-472a-9873-5fab779b18b2"
-					(reference "#PWR091")
-					(unit 1)
-				)
+					(reference "#PWR91")
+					(unit 1)
+				)
