File: Logic_Protection2.kicad_sch (KiCad schematic)
At the start: 10 parts

Commit message: VER2.2: все изменения в списке изменений
Parts:
- D8, D9: value ADM3485E -> ~; Description P/N (none) -> RS485; Product Name (none) -> SN65HVD3082EDR
