File: Driver_1.kicad_sch (KiCad schematic)
At the start: 36 parts

Commit message: VER2.1: добавил схему в доки
Parts:
- renumbered D1 to D31, D1 to D32
Changed lines of the file:
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@@
 (kicad_sch
-	(version 20231120)
+	(version 20250114)
 	(generator "eeschema")
-	(generator_version "8.0")
+	(generator_version "9.0")
 	(paper "A4")
+	(text "Драйвер верхнего ключа"
+		(exclude_from_sim no)
+		(at 71.501 26.543 0)
+		(effects
+			(font
+				(size 1.27 1.27)
+			)
+			(justify left bottom)
+		)
+	)
+	(text "Драйвер нижнего ключа"
+		(exclude_from_sim no)
+		(at 71.247 111.633 0)
+		(effects
+			(font
+				(size 1.27 1.27)
+			)
+			(justify left bottom)
+		)
+	)
+	(text "DESAT Level 1.6V\n650A - 125 C\n900A - 25 C"
+		(exclude_from_sim no)
+		(at 144.145 70.485 0)
+		(effects
+			(font
+				(face "KiCad Font")
+				(size 1.27 1.27)
+			)
+			(justify left)
+		)
+	)
+	(text "DESAT Level 1.6V\n650A - 125 C\n900A - 25 C"
+		(exclude_from_sim no)
+		(at 143.51 121.92 0)
+		(effects
+			(font
+				(face "KiCad Font")
+				(size 1.27 1.27)
+			)
+			(justify left)
+		)
+	)
 	(junction
 		(at 110.49 151.13)
@@
 		)
 	)
-	(text "Драйвер верхнего ключа"
-		(exclude_from_sim no)
-		(at 71.501 26.543 0)
-		(effects
-			(font
-				(size 1.27 1.27)
-			)
-			(justify left bottom)
-		)
-	)
-	(text "Драйвер нижнего ключа"
-		(exclude_from_sim no)
-		(at 71.247 111.633 0)
-		(effects
-			(font
-				(size 1.27 1.27)
-			)
-			(justify left bottom)
-		)
-	)
-	(text "DESAT Level 1.6V\n650A - 125 C\n900A - 25 C"
-		(exclude_from_sim no)
-		(at 144.145 70.485 0)
-		(effects
-			(font
-				(face "KiCad Font")
-				(size 1.27 1.27)
-			)
-			(justify left)
-		)
-	)
-	(text "DESAT Level 1.6V\n650A - 125 C\n900A - 25 C"
-		(exclude_from_sim no)
-		(at 143.51 121.92 0)
-		(effects
-			(font
-				(face "KiCad Font")
-				(size 1.27 1.27)
-			)
-			(justify left)
-		)
-	)
 	(global_label "~{RST_A}"
 		(shape input)
@@
 		(dnp no)
 		(fields_autoplaced yes)
-		(property "Reference" "D1"
+		(property "Reference" "D32"
 			(at 90.17 39.37 0)
 			(effects
@@
 		(dnp no)
 		(fields_autoplaced yes)
-		(property "Reference" "D1"
+		(property "Reference" "D31"
 			(at 90.17 120.65 0)
 			(effects

Commit message: VER2.1: добавил СБ и 3D модели в доки
Other:
- moved on the sheet: C57, C58, C59, C60, C61, C62, C90, C91, D31, D32, D33, D34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
