File: Driver_2.kicad_sch (KiCad schematic)
At the start: 36 parts

Commit message: VER2.1: добавил схему в доки
Parts:
- renumbered D1 to D38, D1 to D64
Changed lines of the file:
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@@
 (kicad_sch
-	(version 20231120)
+	(version 20250114)
 	(generator "eeschema")
-	(generator_version "8.0")
+	(generator_version "9.0")
 	(paper "A4")
+	(text "DESAT Level 1.6V\n650A - 125 C\n900A - 25 C"
+		(exclude_from_sim no)
+		(at 127.635 131.445 0)
+		(effects
+			(font
+				(face "KiCad Font")
+				(size 1.27 1.27)
+			)
+			(justify left)
+		)
+	)
+	(text "Драйвер верхнего ключа"
+		(exclude_from_sim no)
+		(at 71.501 26.543 0)
+		(effects
+			(font
+				(size 1.27 1.27)
+			)
+			(justify left bottom)
+		)
+	)
+	(text "DESAT Level 1.6V\n650A - 125 C\n900A - 25 C"
+		(exclude_from_sim no)
+		(at 146.685 74.295 0)
+		(effects
+			(font
+				(face "KiCad Font")
+				(size 1.27 1.27)
+			)
+			(justify left)
+		)
+	)
+	(text "Драйвер нижнего ключа"
+		(exclude_from_sim no)
+		(at 71.247 111.633 0)
+		(effects
+			(font
+				(size 1.27 1.27)
+			)
+			(justify left bottom)
+		)
+	)
 	(junction
 		(at 123.698 60.96)
@@
 		)
 	)
-	(text "DESAT Level 1.6V\n650A - 125 C\n900A - 25 C"
-		(exclude_from_sim no)
-		(at 127.635 131.445 0)
-		(effects
-			(font
-				(face "KiCad Font")
-				(size 1.27 1.27)
-			)
-			(justify left)
-		)
-	)
-	(text "Драйвер верхнего ключа"
-		(exclude_from_sim no)
-		(at 71.501 26.543 0)
-		(effects
-			(font
-				(size 1.27 1.27)
-			)
-			(justify left bottom)
-		)
-	)
-	(text "DESAT Level 1.6V\n650A - 125 C\n900A - 25 C"
-		(exclude_from_sim no)
-		(at 146.685 74.295 0)
-		(effects
-			(font
-				(face "KiCad Font")
-				(size 1.27 1.27)
-			)
-			(justify left)
-		)
-	)
-	(text "Драйвер нижнего ключа"
-		(exclude_from_sim no)
-		(at 71.247 111.633 0)
-		(effects
-			(font
-				(size 1.27 1.27)
-			)
-			(justify left bottom)
-		)
-	)
 	(global_label "E4"
 		(shape input)
@@
 		(dnp no)
 		(fields_autoplaced yes)
-		(property "Reference" "D1"
+		(property "Reference" "D64"
 			(at 91.44 40.64 0)
 			(effects
@@
 		(dnp no)
 		(fields_autoplaced yes)
-		(property "Reference" "D1"
+		(property "Reference" "D38"
 			(at 91.44 133.35 0)
 			(effects

Commit message: VER2.1: добавил СБ и 3D модели в доки
Other:
- moved on the sheet: C63, C64, C65, C66, C67, C68, C92, C93, D38, D39, D40, D41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
