File: Adapter.kicad_sch (KiCad schematic)
At the start: 0 parts

Commit message: VER2.2.1: исправил все доки
Other:
- note added: "1. Перечень элементов см. НВЦТ.EVP150-2-1.2000.120_v1 ПЭ3."
- note added: "НВЦТ.EVP150-2-1.2000.120_v1"
- note added: "ООО "Электротранспортные"
- note added: "Плата драйверов модуля фазных обмоток"
- note added: "Схема электрическая принципиальная"
- note added: "технологии""
- company: ООО "ЭТТ" -> (none)
- title: Трехфазные драйвера -> (none)
Changed lines of the file:
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@@
 	(paper "A3")
 	(title_block
-		(title "Трехфазные драйвера")
 		(date "2025-06-04")
-		(company "ООО \"ЭТТ\"")
+		(comment 1 "НВЦТ.EVP150-2-1.2000.120_v1 Э3")
 		(comment 2 "Филатов А.С.")
 		(comment 3 "Сизякин А.В.")
+		(comment 4 "Коваленко.В.А.")
+		(comment 6 "Теленков А.П.")
+	)
+	(text "НВЦТ.EVP150-2-1.2000.120_v1"
+		(exclude_from_sim no)
+		(at 16.51 35.56 90)
+		(effects
+			(font
+				(size 2.5 2.5)
+			)
+		)
+	)
+	(text "1. Перечень элементов см. НВЦТ.EVP150-2-1.2000.120_v1 ПЭ3."
+		(exclude_from_sim no)
+		(at 281.432 207.264 0)
+		(effects
+			(font
+				(size 3.5 3.5)
+			)
+		)
+	)
+	(text "технологии\""
+		(exclude_from_sim no)
+		(at 390.906 286.766 0)
+		(effects
+			(font
+				(size 2.5 2.5)
+			)
+		)
+	)
+	(text "ООО \"Электротранспортные"
+		(exclude_from_sim no)
+		(at 389.636 282.702 0)
+		(effects
+			(font
+				(size 2.5 2.5)
+			)
+		)
+	)
+	(text "Схема электрическая принципиальная"
+		(exclude_from_sim no)
+		(at 330.454 271.272 0)
+		(effects
+			(font
+				(size 3 3)
+			)
+		)
+	)
+	(text "Плата драйверов модуля фазных обмоток"
+		(exclude_from_sim no)
+		(at 330.962 264.922 0)
+		(effects
+			(font
+				(size 3 3)
+			)
+		)
 	)
 	(sheet
@@
 			(checksum "9180C2D8C133E7F089AA5E43F4962E04")
 		)
-	)
+		(file
+			(name "gost_portrait.kicad_wks")
+			(type worksheet)
+			(data |KLUv/WC4IM0nAHbqgjFQdTow6/sNILIV1TIw5zlbg/WJMHlF251w3xY6sje8JsLAtpQyyZRKCsq/
+				EmGGgl4DfQBlAHsAvaONk2HUVr50M0HNcN3MsIIB/nRmqIJ0W+eQTWqrbWabxmnwrNvmpduGhqit
+				MpQzDwY4s/OzyailnLl9NEq1BpBGqeohOthGVXIzrLNtPgz0YXqq78ottxDUAZuYGeahqrd6JwUW
+				oqJJqQVJ0BmidgECqIQ22ngYZmcDogKPL3cZ+d2Tcp23ZxrVMvfMDnmdcwcFPMped7nL6B7k73+8
+				I9fr3iO7t2vff9wi5/qSDuM/dH9+7u3L59El7H/s7tit+1/XV8t/vC7CjwIris4vuuj+PfJkGm+m
+				YRSk0W2f3Mf9AWxRqh7RtyGpvx/zvnuMvNdj0smiowXWsWM5qTipVBiO5ssEEy/JUk1MNb4FN5se
+				0eZDLUu48c2vkk6lquGunXRDtS2uWyfVparUUk2pGbW3SbPJ2dEDRkMSEVb7vgWfN6SBEgY4Y7XU
+				i9NKfammWooxyCwVTdpAY2R2AQABlX/kfuztXr/FHSFfTLcoL37r4uV4H0JH8Fi+uN+v0L0TIro7
+				zbQHauVL0Lz3RtDwSjbQPOcLmm15qSUX6UQie+Ti2CWRCFNCuh/kRWeP/bhNdVVgQL6dS0WpLVUF
+				pm7FCaWCvKviRDq5rFTr45ImFeMtGAOBZqgxTalmRJKCpJBhDVGVwBiCmTs7kkAQgjAYQkEcCWIU
+				RFKEKGIIIYQICFHIiJRYO61rAUQ7x+JKGr+IwUgx597QihTG9sWKdeD8KXK0c8VAoma9oCjCMpNB
+				3WiwzwzRt9Bj0pJNf+U2rIYVvomGJkTROrgfqiu5I9YFMgC0gLGuYKO9DqX2aNWWAgZ+GIbl6p2t
+				TQ3qmpxXzXaNf8mD1sEbs+PjnV7IAx+3nLsDFdE7FWcOkVO93DkiijLLTRgdFt1WXBnEDCgpIOow
+				TkehtGrKUgtvcG/QMRQcARw2EVRecM2fx79PY1AHVkzh8wUCcUGI+3mVL6fU9HFHr5NvmGIeJ+ut
+				Q+ZGimF5xjkDNkNeTulEczyWf38ZauM/mTe3ZXjh4GyPcKrBTEVfrRP3AKbd8L2F4YIIAAGMspx2
+				6OxW/zCr9nSI/u5hWdQb1NjExbKDJWWtIQMU11bD3YIRBFxj32kNfuV/HhInKVZ746/3avhEHhiu
+				EturMBRkAsFjLM671UIqKTEf7QfQjYG8dpJtwhUn+qou1NPzKVlhZ+YcpAIkr3TuXG4nOyAcluUv
+				25ZSlkRfwywSaigsWhPn8aJ6ePLSH4kdPH9D/Sz2cEETLR3OvO77gAj4FHZAXlYPWBpgvNpikOLB
+				VAIChSE9wV/3VI6T3ugI+HkgRgnk1ah0Uq7H78lrsrjN7+1j+NjTlP5kFoHueseWhlzPw1uHzhwF
+				sE8Ub87r/mOKKkrVfz55SX9um0mitoeFCgkRV+fPP/NsBIoHHkMLj1YnLLXzkT5nyEpBXE2tCmPZ
+				joyrEqTNYmrhF5bkN7m0miNeQmgetIsG13HsZQjo5eqy4TODonxAp6cWHTBgMuJ1VStPFRnRMJG6
+				2k3V7/45DO9j6WL+KgYD4wM9zutfNtn7hHyN1E8BN0KF64tcysA8pCzjFZz7bVzPtm6AdnnOwUE6
+				GARzhJZzdcgbwiqQD3wkzZ/2DwJqHrgiNBRF5Co=|
+			)
+			(checksum "12F393F2C62B1E595502842B90E2D6BB")
+		)
+	)

Commit message: VER2.2: исправил ошибки в доках
Parts:
- added C10, C3, C31, C36: 10u, Capacitor_SMD:C_1210_3225Metric_Pad1.33x2.70mm_HandSolder, symbol Device:C
- added C37, C38, C4, C9: 4.7u, Capacitor_SMD:C_1206_3216Metric_Pad1.33x1.80mm_HandSolder, symbol Device:C
- added D16, D43: ~, DCDC_My:QA, symbol DCDC_My:QA1
- added L1, L2: 12u, Inductor_SMD:L_1210_3225Metric_Pad1.42x2.65mm_HandSolder, symbol Device:L
- added L7, L8: 47u, Inductor_SMD:L_1812_4532Metric_Pad1.30x3.40mm_HandSolder, symbol Device:L
Connections:
- new net: C37.1, L2.2, L7.1
- new net: C9.1, L1.2, L8.1
- new net: D16.1 (Vin), L8.2
- new net: D43.1 (Vin), L7.2
- new net +15V: C38.1, C4.1, L1.1, L2.1
- new net +15V_H1: C31.1, D43.7 (+Vo)
- new net +15V_L1: C3.1, D16.7 (+Vo)
- new net -15V_H1: C36.2, D43.5 (-Vo)
- new net -15V_L1: C10.2, D16.5 (-Vo)
- new net E1: C31.2, C36.1, D43.6 (0V)
- new net E2: C10.1, C3.2, D16.6 (0V)
- new net GND: C37.2, C38.2, C4.2, C9.2, D16.2 (GND), D43.2 (GND)
Other:
- removed sheet Power_Supply_1
- note added: "1 Перечень элементов см. НВЦТ.EVP150-2-1.2000.120_v1 ПЭ3."
- note added: "Питание драйвера верхнего ключа фазы А"
- note removed: "1. Перечень элементов см. НВЦТ.EVP150-2-1.2000.120_v1 ПЭ3."
